Commit message: 축 뜯어고치는 작업 중

File: urdf/dofbot_for_headlamp.urdf (robot description, URDF)
Before this commit: robot dofbot, 5 links, 4 joints
Links:
- link dofbot_base_link: geometry collision mesh filename=package://smart_headlamp_pkg/meshes/base_link.STL; visual mesh filename=package://smart_headlamp_pkg/meshes/base_link.STL
- link link1: geometry collision mesh filename=package://smart_headlamp_pkg/meshes/link1.STL; visual mesh filename=package://smart_headlamp_pkg/meshes/link1.STL
- link link2: geometry collision mesh filename=package://smart_headlamp_pkg/meshes/link2.STL; visual mesh filename=package://smart_headlamp_pkg/meshes/link2.STL
Joints:
- joint base_link_to_dofbot_base_link: origin xyz=0 0 0 rpy=1.5708 0 1.5708 -> xyz=0 0 0 rpy=-1.5708 0 -1.5708

Commit message: Change meshes to box(sylinder)

File: urdf/dofbot_for_headlamp.urdf (robot description, URDF)
Before this commit: robot dofbot, 5 links, 4 joints
Links:
- removed link marker_link
- added link link3; collision box size=0.042 0.02 0.058; visual box size=0.042 0.02 0.058
- link dofbot_base_link: geometry visual cylinder length=0.005 radius=0.05
- link link1: geometry collision cylinder length=0.04 radius=0.0225; visual cylinder length=0.04 radius=0.0225
- link link2: geometry collision box size=0.03 0.03 0.10; visual box size=0.03 0.03 0.10
Joints:
- removed joint base_link_to_dofbot_base_link
- removed joint marker_joint
- added joint fixed_base_joint: type fixed, parent base_link, child dofbot_base_link, origin xyz=0 0 0 rpy=0 0 0
- added joint joint3: type revolute, parent link2, child link3, origin xyz=0 0 0.08 rpy=0 0 0, axis 0 1 0, limit lower=-1.5708 upper=1.5708 effort=100 velocity=1
- joint joint1: limit lower=-1.5708 upper=1.5708 effort=100 velocity=1 -> (none); origin xyz=0 0 0.064 rpy=0 0 0 -> xyz=0 0 0 rpy=0 0 0; type revolute -> fixed
- joint joint2: axis 0 0 1 -> 1 0 0; origin xyz=0 0 0.0435 rpy=0 1.5708 0 -> xyz=0 0 0.015 rpy=0 0 0

Commit message: Spin link3

File: urdf/dofbot_for_headlamp.urdf (robot description, URDF)
Before this commit: robot dofbot, 5 links, 4 joints
Links:
- link link3: geometry collision box size=0.02 0.042 0.058; visual box size=0.02 0.042 0.058
